Commit message: working version

File: scenes/cyl.urdf.xacro (robot description, xacro)
@@ -18,5 +18,5 @@
   <!-- the gripper -->
   <joint name="map_gripper_joint" type="fixed">
-    <origin xyz="0.0 0.0 0.22" rpy="${M_PI} 0 0"/>
+    <origin xyz="0.0 0.0 0.195" rpy="${M_PI} 0 0"/>
     <parent link="map"/>
     <child link="gripper_mount_link"/>
@@ -56,5 +56,5 @@
   <!-- the graspable object -->
   <joint name="map_graspable_joint" type="floating">
-    <origin xyz="0.0 0.0 0.07" rpy="0 0 0"/>
+    <origin xyz="0.0 0.0 0.05" rpy="0 ${M_PI/2} 0"/>
     <parent link="map"/>
     <child link="graspable"/>
@@ -63,5 +63,5 @@
     <inertial>
       <origin xyz="0.0 0.0 0.0"/>
-      <mass value="0.63352875"/>
+      <mass value="0.0063352875"/>
       <inertia ixx="0.00102103" ixy="0.00000775" ixz="-0.00001230" iyy="0.00080944" iyz="-0.00014417" izz="0.00068788"/>
     </inertial>
@@ -69,5 +69,5 @@
       <origin rpy="0 0 0" xyz="0 0 0"/>
       <geometry>
-        <mesh filename="package://barrett_hand_sim_dart/meshes/cuboid.stl"/>
+        <mesh filename="package://barrett_hand_sim_dart/meshes/cylinder9.stl"/>
       </geometry>
     </visual>
@@ -75,5 +75,5 @@
       <origin rpy="0 0 0" xyz="0 0 0"/>
       <geometry>
-        <mesh filename="package://barrett_hand_sim_dart/meshes/cuboid.stl"/>
+        <mesh filename="package://barrett_hand_sim_dart/meshes/cylinder9.stl"/>
       </geometry>
     </collision>
@@ -81,11 +81,11 @@
   <grasp_specification>
      <init_state joint="right_HandFingerOneKnuckleOneJoint" position="0.01" />
-     <init_state joint="right_HandFingerOneKnuckleTwoJoint" position="0.5" />
-     <init_state joint="right_HandFingerTwoKnuckleTwoJoint" position="0.5" />
-     <init_state joint="right_HandFingerThreeKnuckleTwoJoint" position="0.5" />
+     <init_state joint="right_HandFingerOneKnuckleTwoJoint" position="0.3" />
+     <init_state joint="right_HandFingerTwoKnuckleTwoJoint" position="0.3" />
+     <init_state joint="right_HandFingerThreeKnuckleTwoJoint" position="0.3" />
      <goal_state joint="right_HandFingerOneKnuckleOneJoint" position="0.01" />
-     <goal_state joint="right_HandFingerOneKnuckleTwoJoint" position="1.6" />
-     <goal_state joint="right_HandFingerTwoKnuckleTwoJoint" position="1.6" />
-     <goal_state joint="right_HandFingerThreeKnuckleTwoJoint" position="1.6" />
+     <goal_state joint="right_HandFingerOneKnuckleTwoJoint" position="1.7" />
+     <goal_state joint="right_HandFingerTwoKnuckleTwoJoint" position="1.7" />
+     <goal_state joint="right_HandFingerThreeKnuckleTwoJoint" position="1.7" />
   </grasp_specification>
 </robot>

File: scenes/force.urdf.xacro (robot description, xacro)
@@ -18,5 +18,5 @@
   <!-- the gripper -->
   <joint name="map_gripper_joint" type="fixed">
-    <origin xyz="0.0 0.0 0.22" rpy="${M_PI} 0 0"/>
+    <origin xyz="0.0 0.0 0.195" rpy="${M_PI} 0 0"/>
     <parent link="map"/>
     <child link="gripper_mount_link"/>
@@ -56,5 +56,5 @@
   <!-- the graspable object -->
   <joint name="map_graspable_joint" type="floating">
-    <origin xyz="0.0 0.0 0.07" rpy="0 0 0"/>
+    <origin xyz="0.0 0.0 0.1" rpy="0 ${M_PI/2} 0"/>
     <parent link="map"/>
     <child link="graspable"/>
@@ -63,5 +63,5 @@
     <inertial>
       <origin xyz="0.0 0.0 0.0"/>
-      <mass value="0.63352875"/>
+      <mass value="0.0063352875"/>
       <inertia ixx="0.00102103" ixy="0.00000775" ixz="-0.00001230" iyy="0.00080944" iyz="-0.00014417" izz="0.00068788"/>
     </inertial>
@@ -69,5 +69,5 @@
       <origin rpy="0 0 0" xyz="0 0 0"/>
       <geometry>
-        <mesh filename="package://barrett_hand_sim_dart/meshes/cuboid.stl"/>
+        <mesh filename="package://barrett_hand_sim_dart/meshes/cylinder4.stl"/>
       </geometry>
     </visual>
@@ -75,5 +75,5 @@
       <origin rpy="0 0 0" xyz="0 0 0"/>
       <geometry>
-        <mesh filename="package://barrett_hand_sim_dart/meshes/cuboid.stl"/>
+        <mesh filename="package://barrett_hand_sim_dart/meshes/cylinder4.stl"/>
       </geometry>
     </collision>
@@ -81,11 +81,11 @@
   <grasp_specification>
      <init_state joint="right_HandFingerOneKnuckleOneJoint" position="0.01" />
-     <init_state joint="right_HandFingerOneKnuckleTwoJoint" position="0.5" />
-     <init_state joint="right_HandFingerTwoKnuckleTwoJoint" position="0.5" />
-     <init_state joint="right_HandFingerThreeKnuckleTwoJoint" position="0.5" />
+     <init_state joint="right_HandFingerOneKnuckleTwoJoint" position="1.3" />
+     <init_state joint="right_HandFingerTwoKnuckleTwoJoint" position="1.3" />
+     <init_state joint="right_HandFingerThreeKnuckleTwoJoint" position="1.3" />
      <goal_state joint="right_HandFingerOneKnuckleOneJoint" position="0.01" />
-     <goal_state joint="right_HandFingerOneKnuckleTwoJoint" position="1.6" />
-     <goal_state joint="right_HandFingerTwoKnuckleTwoJoint" position="1.6" />
-     <goal_state joint="right_HandFingerThreeKnuckleTwoJoint" position="1.6" />
+     <goal_state joint="right_HandFingerOneKnuckleTwoJoint" position="2.2" />
+     <goal_state joint="right_HandFingerTwoKnuckleTwoJoint" position="2.2" />
+     <goal_state joint="right_HandFingerThreeKnuckleTwoJoint" position="2.2" />
   </grasp_specification>
 </robot>

File: scenes/sph.urdf.xacro (robot description, xacro)
@@ -18,5 +18,5 @@
   <!-- the gripper -->
   <joint name="map_gripper_joint" type="fixed">
-    <origin xyz="0.0 0.0 0.22" rpy="${M_PI} 0 0"/>
+    <origin xyz="0.0 0.0 0.21" rpy="${M_PI} 0 0"/>
     <parent link="map"/>
     <child link="gripper_mount_link"/>
@@ -56,5 +56,5 @@
   <!-- the graspable object -->
   <joint name="map_graspable_joint" type="floating">
-    <origin xyz="0.0 0.0 0.07" rpy="0 0 0"/>
+    <origin xyz="0.0 0.0 0.05" rpy="0 0 0"/>
     <parent link="map"/>
     <child link="graspable"/>
@@ -63,5 +63,5 @@
     <inertial>
       <origin xyz="0.0 0.0 0.0"/>
-      <mass value="0.63352875"/>
+      <mass value="0.0063352875"/>
       <inertia ixx="0.00102103" ixy="0.00000775" ixz="-0.00001230" iyy="0.00080944" iyz="-0.00014417" izz="0.00068788"/>
     </inertial>
@@ -69,5 +69,5 @@
       <origin rpy="0 0 0" xyz="0 0 0"/>
       <geometry>
-        <mesh filename="package://barrett_hand_sim_dart/meshes/cuboid.stl"/>
+        <mesh filename="package://barrett_hand_sim_dart/meshes/cylinder6.stl"/>
       </geometry>
     </visual>
@@ -75,17 +75,17 @@
       <origin rpy="0 0 0" xyz="0 0 0"/>
       <geometry>
-        <mesh filename="package://barrett_hand_sim_dart/meshes/cuboid.stl"/>
+        <mesh filename="package://barrett_hand_sim_dart/meshes/cylinder6.stl"/>
       </geometry>
     </collision>
   </link>
   <grasp_specification>
-     <init_state joint="right_HandFingerOneKnuckleOneJoint" position="0.01" />
-     <init_state joint="right_HandFingerOneKnuckleTwoJoint" position="0.5" />
-     <init_state joint="right_HandFingerTwoKnuckleTwoJoint" position="0.5" />
-     <init_state joint="right_HandFingerThreeKnuckleTwoJoint" position="0.5" />
-     <goal_state joint="right_HandFingerOneKnuckleOneJoint" position="0.01" />
-     <goal_state joint="right_HandFingerOneKnuckleTwoJoint" position="1.6" />
-     <goal_state joint="right_HandFingerTwoKnuckleTwoJoint" position="1.6" />
-     <goal_state joint="right_HandFingerThreeKnuckleTwoJoint" position="1.6" />
+     <init_state joint="right_HandFingerOneKnuckleOneJoint" position="1.0" />
+     <init_state joint="right_HandFingerOneKnuckleTwoJoint" position="0.9" />
+     <init_state joint="right_HandFingerTwoKnuckleTwoJoint" position="0.9" />
+     <init_state joint="right_HandFingerThreeKnuckleTwoJoint" position="0.3" />
+     <goal_state joint="right_HandFingerOneKnuckleOneJoint" position="1.0" />
+     <goal_state joint="right_HandFingerOneKnuckleTwoJoint" position="1.7" />
+     <goal_state joint="right_HandFingerTwoKnuckleTwoJoint" position="1.7" />
+     <goal_state joint="right_HandFingerThreeKnuckleTwoJoint" position="1.7" />
   </grasp_specification>
 </robot>
