Commit message: experiments ok

File: scenes/test_container_1.urdf.xacro (robot description, xacro)
@@ -56,5 +56,5 @@
   <!-- the graspable object -->
   <joint name="map_graspable_joint" type="floating">
-    <origin xyz="0.0 0.0 0.2" rpy="0 0 0"/>
+    <origin xyz="0.0 0.0 0.1" rpy="0 0 0"/>
     <parent link="map"/>
     <child link="graspable"/>

File: scenes/test_container_2.urdf.xacro (robot description, xacro)
@@ -56,5 +56,5 @@
   <!-- the graspable object -->
   <joint name="map_graspable_joint" type="floating">
-    <origin xyz="0.0 0.0 0.2" rpy="0 0 0"/>
+    <origin xyz="0.0 0.0 0.1" rpy="0 0 0"/>
     <parent link="map"/>
     <child link="graspable"/>

File: scenes/test_cuboid.urdf.xacro (robot description, xacro)
@@ -56,5 +56,5 @@
   <!-- the graspable object -->
   <joint name="map_graspable_joint" type="floating">
-    <origin xyz="0.0 0.0 0.2" rpy="0 0 0"/>
+    <origin xyz="0.0 0.0 0.1" rpy="0 0 0"/>
     <parent link="map"/>
     <child link="graspable"/>
