Commit message: experiments

File: objects/container_1d.urdf (robot description, URDF)
Before this commit: robot object, 2 links, 1 joints
Links:
- removed link object
- added link graspable, mass 0.63352875; collision mesh filename=package://barrett_hand_sim_dart/meshes/container_1d.stl; visual mesh filename=package://barrett_hand_sim_dart/meshes/container_1d.stl
Joints:
- joint arm_world_joint: child object -> graspable

File: objects/container_2d.urdf (robot description, URDF)
Before this commit: robot object, 2 links, 1 joints
Links:
- removed link object
- added link graspable, mass 0.63352875; collision mesh filename=package://barrett_hand_sim_dart/meshes/container_2d.stl; visual mesh filename=package://barrett_hand_sim_dart/meshes/container_2d.stl
Joints:
- joint arm_world_joint: child object -> graspable

File: objects/cube.urdf (robot description, URDF)
Before this commit: robot cube5, 2 links, 1 joints
Links:
- removed link cube5
- added link graspable, mass 0.63352875; collision mesh filename=package://barrett_hand_sim_dart/meshes/cuboid.stl; visual mesh filename=package://barrett_hand_sim_dart/meshes/cuboid.stl
Joints:
- joint arm_world_joint: child cube5 -> graspable

File: objects/cylinder4.urdf (robot description, URDF)
Before this commit: robot cube5, 2 links, 1 joints
Links:
- removed link cube5
- added link graspable, mass 0.63352875; collision mesh filename=package://barrett_hand_sim_dart/meshes/cylinder4.stl; visual mesh filename=package://barrett_hand_sim_dart/meshes/cylinder4.stl
Joints:
- joint arm_world_joint: child cube5 -> graspable

File: objects/jar.urdf (robot description, URDF)
Before this commit: robot cylinder9, 2 links, 1 joints
Links:
- removed link cylinder9
- added link graspable, mass 0.63352875; collision mesh filename=package://barrett_hand_sim_dart/meshes/cylinder9.stl; visual mesh filename=package://barrett_hand_sim_dart/meshes/cylinder9.stl
Joints:
- joint arm_world_joint: child cylinder9 -> graspable

File: objects/jar2.urdf (robot description, URDF)
Before this commit: robot cylinder6, 2 links, 1 joints
Links:
- removed link cylinder6
- added link graspable, mass 0.63352875; collision mesh filename=package://barrett_hand_sim_dart/meshes/cylinder6.stl; visual mesh filename=package://barrett_hand_sim_dart/meshes/cylinder6.stl
Joints:
- joint arm_world_joint: child cylinder6 -> graspable

File: objects/kettle15d.urdf (robot description, URDF)
Before this commit: robot object, 2 links, 1 joints
Links:
- removed link object
- added link graspable, mass 0.63352875; collision mesh filename=package://barrett_hand_sim_dart/meshes/kettle15d.stl; visual mesh filename=package://barrett_hand_sim_dart/meshes/kettle15d.stl
Joints:
- joint arm_world_joint: child object -> graspable

File: objects/mug.urdf (robot description, URDF)
Before this commit: robot object, 2 links, 1 joints
Links:
- removed link object
- added link graspable, mass 0.63352875; collision mesh filename=package://barrett_hand_sim_dart/meshes/cyl_w_closed_handle.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; visual mesh filename=package://barrett_hand_sim_dart/meshes/cyl_w_closed_handle.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
Joints:
- joint arm_world_joint: child object -> graspable
